File: schematics/SCHv2.brd (EAGLE design)
At the start: 23.5 x 39.4 mm, 11 parts, among them J2 POWER_JACKSLT, Q3 TIP31C

Commit message: fixing wiring (power jack)
turns out the ground of the power jack was swapped with the signal pin on the jack, all fixed in this push. sadly I have 10 boards with this issue, easy fix though. 👍
Connections:
- net N$4: now also J2.GND@1; no longer J2.GND@2
Routing:
- net N$4: track 33.0 -> 41.9 mm
Changed lines of the file:
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@@
 <drawing>
 <settings>
-<setting alwaysvectorfont="yes"/>
+<setting alwaysvectorfont="no"/>
 <setting verticaltext="up"/>
 </settings>
@@
 <wire x1="31.75" y1="50.8" x2="31.75" y2="52.07" width="0.6096" layer="1"/>
 <wire x1="31.75" y1="52.07" x2="36.83" y2="57.15" width="0.6096" layer="1"/>
-<wire x1="34.925" y1="64.77" x2="34.925" y2="63.8175" width="0.6096" layer="1"/>
+<wire x1="34.925" y1="64.77" x2="34.925" y2="64.135" width="0.6096" layer="1"/>
 <wire x1="34.925" y1="64.135" x2="34.925" y2="63.8175" width="0.6096" layer="1"/>
-<wire x1="34.925" y1="64.135" x2="34.925" y2="59.055" width="0.6096" layer="1"/>
+<wire x1="34.925" y1="63.8175" x2="34.925" y2="59.055" width="0.6096" layer="1"/>
 <wire x1="34.925" y1="59.055" x2="36.83" y2="57.15" width="0.6096" layer="1"/>
-<contactref element="J2" pad="GND@2"/>
-<wire x1="38.4575" y1="64.13" x2="34.93" y2="64.13" width="0.6096" layer="1"/>
 <wire x1="34.93" y1="64.13" x2="34.925" y2="64.135" width="0.6096" layer="1"/>
 <wire x1="33.655" y1="66.04" x2="34.925" y2="64.77" width="0.6096" layer="1"/>
+<contactref element="J2" pad="GND@1"/>
+<wire x1="36.83" y1="57.15" x2="40.3225" y2="60.6425" width="0.6096" layer="1"/>
+<wire x1="40.3225" y1="60.6425" x2="40.3225" y2="64.295" width="0.6096" layer="1"/>
+<wire x1="40.3225" y1="64.295" x2="43.4575" y2="67.43" width="0.6096" layer="1"/>
 </signal>
 <signal name="N$7">
